File: pcb-main-nautilus-atmega4809-sheet-bi_directional_level_shifter.kicad_sch (KiCad schematic)
At the start: 3 parts, among them Q1 BSS138PW,115

Commit message: Switch to generated Digi-Key and Mouser links
Supports #2.
Parts:
- Q1: Digi-Key https://www.digikey.com/en/products/detail/nexperia-usa-inc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 -> (none); Digi-Key Part Number (none) -> 1727-1143-1-ND; Mouser https://www.mouser.com/ProductDetail/Nexperia/BSS138PW115?q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 -> (none); Mouser Part Number (none) -> 771-BSS138PW115
- R5, R6: Digi-Key https://www.digikey.com/en/products/detail/panasonic-electr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 -> (none); Digi-Key Part Number (none) -> P4.70KHCT-ND; Mouser https://www.mouser.com/ProductDetail/Panasonic/ERJ-3EKF4701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 -> (none); Mouser Part Number (none) -> 667-ERJ-3EKF4701V
Changed lines of the file:
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@@
       (effects (font (size 1.27 1.27)) hide)
     )
-    (property "Digi-Key" "https://www.digikey.com/en/products/detail/panasonic-electronic-components/ERJ-3EKF4701V/1746419" (id 6) (at 154.94 105.41 0)
+    (property "Digi-Key Part Number" "P4.70KHCT-ND" (id 6) (at 154.94 105.41 0)
       (effects (font (size 1.27 1.27)) hide)
     )
-    (property "Mouser" "https://www.mouser.com/ProductDetail/Panasonic/ERJ-3EKF4701V?qs=MVjVSMjNRMouVvwnqrpO2w%3D%3D" (id 7) (at 154.94 105.41 0)
+    (property "Mouser Part Number" "667-ERJ-3EKF4701V" (id 7) (at 154.94 105.41 0)
       (effects (font (size 1.27 1.27)) hide)
     )
@@
       (effects (font (size 1.27 1.27)) hide)
     )
-    (property "Digi-Key" "https://www.digikey.com/en/products/detail/panasonic-electronic-components/ERJ-3EKF4701V/1746419" (id 6) (at 124.46 105.41 0)
+    (property "Digi-Key Part Number" "P4.70KHCT-ND" (id 6) (at 124.46 105.41 0)
       (effects (font (size 1.27 1.27)) hide)
     )
-    (property "Mouser" "https://www.mouser.com/ProductDetail/Panasonic/ERJ-3EKF4701V?qs=MVjVSMjNRMouVvwnqrpO2w%3D%3D" (id 7) (at 124.46 105.41 0)
+    (property "Mouser Part Number" "667-ERJ-3EKF4701V" (id 7) (at 124.46 105.41 0)
       (effects (font (size 1.27 1.27)) hide)
     )
@@
       (effects (font (size 1.27 1.27)) hide)
     )
-    (property "Digi-Key" "https://www.digikey.com/en/products/detail/nexperia-usa-inc/BSS138PW-115/2779826" (id 6) (at 139.7 107.95 90)
+    (property "Digi-Key Part Number" "1727-1143-1-ND" (id 6) (at 139.7 107.95 90)
       (effects (font (size 1.27 1.27)) hide)
     )
-    (property "Mouser" "https://www.mouser.com/ProductDetail/Nexperia/BSS138PW115?qs=A1cBxND5mHKdv5mYHLzmBw%3D%3D" (id 7) (at 139.7 107.95 90)
+    (property "Mouser Part Number" "771-BSS138PW115" (id 7) (at 139.7 107.95 90)
       (effects (font (size 1.27 1.27)) hide)
     )

Commit message: Replace Digi-Key part numbers with links
Supports #2.
Parts:
- Q1: Digi-Key (none) -> https://www.digikey.com/en/products/detail/nexperia-usa-inc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; Digi-Key Part Number 1727-1143-1-ND -> (none)
- R5, R6: Digi-Key (none) -> https://www.digikey.com/en/products/detail/panasonic-electr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; Digi-Key Part Number P4.70KHCT-ND -> (none)
Changed lines of the file:
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@@
       (effects (font (size 1.27 1.27)) hide)
     )
-    (property "Digi-Key Part Number" "P4.70KHCT-ND" (id 6) (at 154.94 105.41 0)
+    (property "Digi-Key" "https://www.digikey.com/en/products/detail/panasonic-electronic-components/ERJ-3EKF4701V/1746419" (id 6) (at 154.94 105.41 0)
       (effects (font (size 1.27 1.27)) hide)
     )
@@
       (effects (font (size 1.27 1.27)) hide)
     )
-    (property "Digi-Key Part Number" "P4.70KHCT-ND" (id 6) (at 124.46 105.41 0)
+    (property "Digi-Key" "https://www.digikey.com/en/products/detail/panasonic-electronic-components/ERJ-3EKF4701V/1746419" (id 6) (at 124.46 105.41 0)
       (effects (font (size 1.27 1.27)) hide)
     )
@@
       (effects (font (size 1.27 1.27)) hide)
     )
-    (property "Digi-Key Part Number" "1727-1143-1-ND" (id 6) (at 139.7 107.95 90)
+    (property "Digi-Key" "https://www.digikey.com/en/products/detail/nexperia-usa-inc/BSS138PW-115/2779826" (id 6) (at 139.7 107.95 90)
       (effects (font (size 1.27 1.27)) hide)
     )

Commit message: Replace Mouser part numbers with links
Supports #2.
Parts:
- Q1: Mouser (none) -> https://www.mouser.com/ProductDetail/Nexperia/BSS138PW115?q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; Mouser Part Number 771-BSS138PW115 -> (none)
- R5, R6: Mouser (none) -> https://www.mouser.com/ProductDetail/Panasonic/ERJ-3EKF4701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; Mouser Part Number 667-ERJ-3EKF4701V -> (none)
Changed lines of the file:
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@@
       (effects (font (size 1.27 1.27)) hide)
     )
-    (property "Mouser Part Number" "667-ERJ-3EKF4701V" (id 7) (at 154.94 105.41 0)
+    (property "Mouser" "https://www.mouser.com/ProductDetail/Panasonic/ERJ-3EKF4701V?qs=MVjVSMjNRMouVvwnqrpO2w%3D%3D" (id 7) (at 154.94 105.41 0)
       (effects (font (size 1.27 1.27)) hide)
     )
@@
       (effects (font (size 1.27 1.27)) hide)
     )
-    (property "Mouser Part Number" "667-ERJ-3EKF4701V" (id 7) (at 124.46 105.41 0)
+    (property "Mouser" "https://www.mouser.com/ProductDetail/Panasonic/ERJ-3EKF4701V?qs=MVjVSMjNRMouVvwnqrpO2w%3D%3D" (id 7) (at 124.46 105.41 0)
       (effects (font (size 1.27 1.27)) hide)
     )
@@
       (effects (font (size 1.27 1.27)) hide)
     )
-    (property "Mouser Part Number" "771-BSS138PW115" (id 7) (at 139.7 107.95 90)
+    (property "Mouser" "https://www.mouser.com/ProductDetail/Nexperia/BSS138PW115?qs=A1cBxND5mHKdv5mYHLzmBw%3D%3D" (id 7) (at 139.7 107.95 90)
       (effects (font (size 1.27 1.27)) hide)
     )
