File: pcb-main-nautilus-atmega4809-sheet-mcu.kicad_sch (KiCad schematic)
At the start: 10 parts

Commit message: Annotate schematic
Supports #2.
Parts:
- gave numbers to parts that had none: 10
Changed lines of the file:
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@@
   (symbol (lib_id "MCU_Microchip_ATmega:ATmega4809-A") (at 139.7 107.95 0) (unit 1)
     (in_bom yes) (on_board yes) (fields_autoplaced)
-    (property "Reference" "U?" (id 0) (at 141.7194 143.51 0)
+    (property "Reference" "U4" (id 0) (at 141.7194 143.51 0)
       (effects (font (size 1.27 1.27)) (justify left))
     )
@@
   (symbol (lib_id "Device:C_Small") (at 111.76 140.97 0) (unit 1)
     (in_bom yes) (on_board yes) (fields_autoplaced)
-    (property "Reference" "C?" (id 0) (at 114.3 139.7062 0)
+    (property "Reference" "C16" (id 0) (at 114.3 139.7062 0)
       (effects (font (size 1.27 1.27)) (justify left))
     )
@@
   (symbol (lib_id "Device:C_Small") (at 149.86 64.77 270) (unit 1)
     (in_bom yes) (on_board yes) (fields_autoplaced)
-    (property "Reference" "C?" (id 0) (at 149.8536 58.42 90))
+    (property "Reference" "C14" (id 0) (at 149.8536 58.42 90))
     (property "Value" "0.1uF/10V" (id 1) (at 149.8536 60.96 90))
     (property "Footprint" "Capacitor_SMD:C_0603_1608Metric_Pad1.08x0.95mm_HandSolder" (id 2) (at 149.86 64.77 0)
@@
   (symbol (lib_id "Device:C_Small") (at 132.08 64.77 270) (unit 1)
     (in_bom yes) (on_board yes) (fields_autoplaced)
-    (property "Reference" "C?" (id 0) (at 132.0736 58.42 90))
+    (property "Reference" "C13" (id 0) (at 132.0736 58.42 90))
     (property "Value" "0.1uF/10V" (id 1) (at 132.0736 60.96 90))
     (property "Footprint" "Capacitor_SMD:C_0603_1608Metric_Pad1.08x0.95mm_HandSolder" (id 2) (at 132.08 64.77 0)
@@
   (symbol (lib_id "Device:C_Small") (at 96.52 140.97 0) (unit 1)
     (in_bom yes) (on_board yes) (fields_autoplaced)
-    (property "Reference" "C?" (id 0) (at 99.06 139.7062 0)
+    (property "Reference" "C15" (id 0) (at 99.06 139.7062 0)
       (effects (font (size 1.27 1.27)) (justify left))
     )
@@
   (symbol (lib_id "Device:NetTie_3") (at 203.2 76.2 0) (unit 1)
     (in_bom no) (on_board yes) (fields_autoplaced)
-    (property "Reference" "NT?" (id 0) (at 203.2 71.12 0))
+    (property "Reference" "NT2" (id 0) (at 203.2 71.12 0))
     (property "Value" "NetTie_3" (id 1) (at 203.2 73.66 0))
     (property "Footprint" "" (id 2) (at 203.2 76.2 0)
@@
   (symbol (lib_id "Device:NetTie_3") (at 203.2 88.9 0) (unit 1)
     (in_bom no) (on_board yes) (fields_autoplaced)
-    (property "Reference" "NT?" (id 0) (at 203.2 83.82 0))
+    (property "Reference" "NT3" (id 0) (at 203.2 83.82 0))
     (property "Value" "NetTie_3" (id 1) (at 203.2 86.36 0))
     (property "Footprint" "" (id 2) (at 203.2 88.9 0)
@@
   (symbol (lib_id "Device:C_Small") (at 132.08 54.61 270) (unit 1)
     (in_bom yes) (on_board yes) (fields_autoplaced)
-    (property "Reference" "C?" (id 0) (at 132.0736 48.26 90))
+    (property "Reference" "C11" (id 0) (at 132.0736 48.26 90))
     (property "Value" "0.1uF/10V" (id 1) (at 132.0736 50.8 90))
     (property "Footprint" "Capacitor_SMD:C_0603_1608Metric_Pad1.08x0.95mm_HandSolder" (id 2) (at 132.08 54.61 0)
@@
   (symbol (lib_id "Device:C_Small") (at 132.08 44.45 270) (unit 1)
     (in_bom yes) (on_board yes) (fields_autoplaced)
-    (property "Reference" "C?" (id 0) (at 132.0736 38.1 90))
+    (property "Reference" "C10" (id 0) (at 132.0736 38.1 90))
     (property "Value" "4.7uF/10V" (id 1) (at 132.0736 40.64 90))
     (property "Footprint" "Capacitor_SMD:C_0603_1608Metric_Pad1.08x0.95mm_HandSolder" (id 2) (at 132.08 44.45 0)
@@
   (symbol (lib_id "Device:C_Small") (at 149.86 54.61 270) (unit 1)
     (in_bom yes) (on_board yes) (fields_autoplaced)
-    (property "Reference" "C?" (id 0) (at 149.8536 48.26 90))
+    (property "Reference" "C12" (id 0) (at 149.8536 48.26 90))
     (property "Value" "4.7uF/10V" (id 1) (at 149.8536 50.8 90))
     (property "Footprint" "Capacitor_SMD:C_0603_1608Metric_Pad1.08x0.95mm_HandSolder" (id 2) (at 149.86 54.61 0)

Commit message: Add nettie footprints
Supports #2.
Parts:
- NT2, NT3: footprint (none) -> NetTie:NetTie-3_SMD_Pad0.5mm
Changed lines of the file:
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@@
     (property "Reference" "NT2" (id 0) (at 203.2 71.12 0))
     (property "Value" "NetTie_3" (id 1) (at 203.2 73.66 0))
-    (property "Footprint" "" (id 2) (at 203.2 76.2 0)
+    (property "Footprint" "NetTie:NetTie-3_SMD_Pad0.5mm" (id 2) (at 203.2 76.2 0)
       (effects (font (size 1.27 1.27)) hide)
     )
@@
     (property "Reference" "NT3" (id 0) (at 203.2 83.82 0))
     (property "Value" "NetTie_3" (id 1) (at 203.2 86.36 0))
-    (property "Footprint" "" (id 2) (at 203.2 88.9 0)
+    (property "Footprint" "NetTie:NetTie-3_SMD_Pad0.5mm" (id 2) (at 203.2 88.9 0)
       (effects (font (size 1.27 1.27)) hide)
     )

Commit message: Add D13 LED
Supports #2.
Parts:
- added D5: RED, LED_SMD:LED_0603_1608Metric_Pad1.05x0.95mm_HandSolder, symbol Device:LED_Small
- added R11: 330/0.1W, Resistor_SMD:R_0603_1608Metric_Pad0.98x0.95mm_HandSolder, symbol Device:R_Small
Connections:
- net D13/SCK: now also D5.2 (A)
- net GND: now also R11.2
- new net: D5.1 (K), R11.1
Changed lines of the file:
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@@
+    (stroke (width 0) (type default) (color 0 0 0 0))
+  )
+  (wire (pts (xy 200.66 101.6) (xy 203.2 101.6))
+    (stroke (width 0) (type default) (color 0 0 0 0))
+  )
+  (wire (pts (xy 203.2 101.6) (xy 203.2 104.14))
     (stroke (width 0) (type default) (color 0 0 0 0))
   )
@@
     (stroke (width 0) (type default) (color 0 0 0 0))
   )
+  (wire (pts (xy 203.2 116.84) (xy 203.2 119.38))
+    (stroke (width 0) (type default) (color 0 0 0 0))
+  )
   (wire (pts (xy 134.62 44.45) (xy 139.7 44.45))
     (stroke (width 0) (type default) (color 0 0 0 0))
   )
   (wire (pts (xy 157.48 54.61) (xy 157.48 64.77))
+    (stroke (width 0) (type default) (color 0 0 0 0))
+  )
+  (wire (pts (xy 203.2 109.22) (xy 203.2 111.76))
     (stroke (width 0) (type default) (color 0 0 0 0))
   )
@@
     (effects (font (size 1.27 1.27)) (justify right))
   )
+  (hierarchical_label "D13{slash}SCK" (shape bidirectional) (at 200.66 101.6 180)
+    (effects (font (size 1.27 1.27)) (justify right))
+  )
   (hierarchical_label "D18{slash}A4{slash}SDA" (shape bidirectional) (at 208.28 76.2 0)
     (effects (font (size 1.27 1.27)) (justify left))
@@
   (hierarchical_label "HOST_TX" (shape bidirectional) (at 157.48 110.49 0)
     (effects (font (size 1.27 1.27)) (justify left))
+  )
+  (hierarchical_label "GND" (shape input) (at 203.2 119.38 270)
+    (effects (font (size 1.27 1.27)) (justify right))
+  )
+  (symbol (lib_id "Device:R_Small") (at 203.2 114.3 0) (unit 1)
+    (in_bom yes) (on_board yes) (fields_autoplaced)
+    (property "Reference" "R11" (id 0) (at 205.74 113.0299 0)
+      (effects (font (size 1.27 1.27)) (justify left))
+    )
+    (property "Value" "330/0.1W" (id 1) (at 205.74 115.5699 0)
+      (effects (font (size 1.27 1.27)) (justify left))
+    )
+    (property "Footprint" "Resistor_SMD:R_0603_1608Metric_Pad0.98x0.95mm_HandSolder" (id 2) (at 203.2 114.3 0)
+      (effects (font (size 1.27 1.27)) hide)
+    )
+    (property "Datasheet" "https://industrial.panasonic.com/cdbs/www-data/pdf/RDA0000/AOA0000C304.pdf" (id 3) (at 203.2 114.3 0)
+      (effects (font (size 1.27 1.27)) hide)
+    )
+    (property "Manufacturer" "Panasonic Electronic Components" (id 4) (at 203.2 114.3 0)
+      (effects (font (size 1.27 1.27)) hide)
+    )
+    (property "Manufacturer Part Number" "ERJ-3EKF3300V" (id 5) (at 203.2 114.3 0)
+      (effects (font (size 1.27 1.27)) hide)
+    )
+    (property "Digi-Key" "https://www.digikey.com/en/products/detail/panasonic-electronic-components/ERJ-3EKF3300V/1746374" (id 6) (at 203.2 114.3 0)
+      (effects (font (size 1.27 1.27)) hide)
+    )
+    (property "Mouser" "https://www.mouser.com/ProductDetail/Panasonic/ERJ-3EKF3300V?qs=MVjVSMjNRMqskx0rzM4%2FYg%3D%3D" (id 7) (at 203.2 114.3 0)
+      (effects (font (size 1.27 1.27)) hide)
+    )
+    (pin "1")
+    (pin "2")
   )
   (symbol (lib_id "MCU_Microchip_ATmega:ATmega4809-A") (at 139.7 107.95 0) (unit 1)
@@
     (pin "3")
   )
+  (symbol (lib_id "Device:LED_Small") (at 203.2 106.68 90) (unit 1)
+    (in_bom yes) (on_board yes) (fields_autoplaced)
+    (property "Reference" "D5" (id 0) (at 205.74 105.3464 90)
+      (effects (font (size 1.27 1.27)) (justify right))
+    )
+    (property "Value" "RED" (id 1) (at 205.74 107.8864 90)
+      (effects (font (size 1.27 1.27)) (justify right))
+    )
+    (property "Footprint" "LED_SMD:LED_0603_1608Metric_Pad1.05x0.95mm_HandSolder" (id 2) (at 203.2 106.68 90)
+      (effects (font (size 1.27 1.27)) hide)
+    )
+    (property "Datasheet" "https://optoelectronics.liteon.com/upload/download/DS-22-99-0151/LTST-C190KRKT.pdf" (id 3) (at 203.2 106.68 90)
+      (effects (font (size 1.27 1.27)) hide)
+    )
+    (property "Manufacturer" "Lite-On Inc." (id 4) (at 203.2 106.68 90)
+      (effects (font (size 1.27 1.27)) hide)
+    )
+    (property "Manufacturer Part Number" "LTST-C190KRKT" (id 5) (at 203.2 106.68 90)
+      (effects (font (size 1.27 1.27)) hide)
+    )
+    (property "Digi-Key" "https://www.digikey.com/en/products/detail/liteon/LTST-C190KRKT/386817" (id 6) (at 203.2 106.68 90)
+      (effects (font (size 1.27 1.27)) hide)
+    )
+    (property "Mouser" "https://www.mouser.com/ProductDetail/Lite-On/LTST-C190KRKT?qs=kAD5fFa1n5VY3YYNWPC1Fg%3D%3D" (id 7) (at 203.2 106.68 90)
+      (effects (font (size 1.27 1.27)) hide)
+    )
+    (pin "1")
+    (pin "2")
+  )
   (symbol (lib_id "Device:C_Small") (at 132.08 54.61 270) (unit 1)

Commit message: Add serial LEDs
Supports #2.
Parts:
- added D5, D7: YELLOW, LED_SMD:LED_0603_1608Metric_Pad1.05x0.95mm_HandSolder, symbol Device:LED_Small
- added R11, R13: 330/0.1W, Resistor_SMD:R_0603_1608Metric_Pad0.98x0.95mm_HandSolder, symbol Device:R_Small
- renumbered D5 to D6, R11 to R12
Connections:
- net GND: now also R11.2, R13.2
- net HOST_RX: now also D7.2 (A)
- net HOST_TX: now also D5.2 (A)
- new net: D5.1 (K), R11.1
- new net: D7.1 (K), R13.1

Commit message: Add MCU reset circuit
Supports #2.
Parts:
- added C15: 0.1uF/10V, Capacitor_SMD:C_0603_1608Metric_Pad1.08x0.95mm_HandSolder, symbol Device:C_Small
- added R11: 4.7k/0.1W, Resistor_SMD:R_0603_1608Metric_Pad0.98x0.95mm_HandSolder, symbol Device:R_Small
- added R12: 330/0.1W, Resistor_SMD:R_0603_1608Metric_Pad0.98x0.95mm_HandSolder, symbol Device:R_Small
- added SW1: PTS645SH43SMTR92 LFS, Button_Switch_SMD:SW_Push_1P1T_NO_6x6mm_H9.5mm, symbol Switch:SW_Push
- renumbered C15 to C16, C16 to C17, D6 to D5, D5 to D6, R12 to R13, R11 to R14, R13 to R15
Connections:
- net 5V: now also R11.1
- net GND: now also C15.2, SW1.1
- net ~{RESET}: now also C15.1, R11.2, R12.2
- new net: R12.1, SW1.2
Other:
- moved on the sheet: D6, D7, R14, R15

Commit message: Switch to generated Digi-Key and Mouser links
Supports #2.
Parts:
- C10, C12, C16: Digi-Key https://www.digikey.com/en/products/detail/kemet/C0603C475M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 -> (none); Digi-Key Part Number (none) -> 399-C0603C475M8PAC7867CT-ND; Mouser https://www.mouser.com/ProductDetail/KEMET/C0603C106M9PAC?q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 -> (none); Mouser Part Number (none) -> 80-C0603C106M9PAC
- C11, C13, C14, C15, C17: Digi-Key https://www.digikey.com/en/products/detail/kemet/C0603C104M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 -> (none); Digi-Key Part Number (none) -> 399-C0603C104M8RAC7867CT-ND; Mouser https://www.mouser.com/ProductDetail/KEMET/C0603C104M8RACTU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 -> (none); Mouser Part Number (none) -> 80-C0603C104M8R
- D5: Digi-Key https://www.digikey.com/en/products/detail/liteon/LTST-C190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 -> (none); Digi-Key Part Number (none) -> 160-1436-1-ND; Mouser https://www.mouser.com/ProductDetail/Lite-On/LTST-C190KRKT?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 -> (none); Mouser Part Number (none) -> 859-LTST-C190KRKT
- D6, D7: Digi-Key https://www.digikey.com/en/products/detail/liteon/LTST-C190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 -> (none); Digi-Key Part Number (none) -> 160-1437-1-ND; Mouser https://www.mouser.com/ProductDetail/Lite-On/LTST-C190KSKT?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 -> (none); Mouser Part Number (none) -> 859-LTST-C190KSKT
- R11: Digi-Key https://www.digikey.com/en/products/detail/panasonic-electr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 -> (none); Digi-Key Part Number (none) -> P4.70KHCT-ND; Mouser https://www.mouser.com/ProductDetail/Panasonic/ERJ-3EKF4701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 -> (none); Mouser Part Number (none) -> 667-ERJ-3EKF4701V
- R12, R13, R14, R15: Digi-Key https://www.digikey.com/en/products/detail/panasonic-electr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 -> (none); Digi-Key Part Number (none) -> P330HCT-ND; Mouser https://www.mouser.com/ProductDetail/Panasonic/ERJ-3EKF3300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 -> (none); Mouser Part Number (none) -> 667-ERJ-3EKF3300V
- SW1: Digi-Key https://www.digikey.com/en/products/detail/c-k/PTS645SH43SM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 -> (none); Digi-Key Part Number (none) -> CKN11907CT-ND; Field7 https://www.mouser.com/ProductDetail/CK/PTS645SH43SMTR92LFS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 -> (none); Mouser Part Number (none) -> 611-PTS645SH43SMTR92
- U4: Digi-Key Part Number (none) -> 150-ATMEGA4809-AURCT-ND; Manufacturer (none) -> Microchip Technology; Manufacturer Part Number (none) -> ATMEGA4809-AU; Mouser Part Number (none) -> 556-ATMEGA4809-AUR
