File: pcb-main-nautilus-atmega4809-sheet-power.kicad_sch (KiCad schematic)
At the start: 14 parts, among them U1 NCP1117-5.0_TO252, U2 AP2112K-3.3

Commit message: Add electrolytic capacitor footprints
Supports #2.
Parts:
- C1: footprint (none) -> Capacitor_SMD:CP_Elec_6.3x7.7
- C3: footprint (none) -> Capacitor_SMD:CP_Elec_4x5.8
Changed lines of the file:
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@@
       (effects (font (size 1.27 1.27)) (justify left))
     )
-    (property "Footprint" "" (id 2) (at 101.6 74.93 0)
+    (property "Footprint" "Capacitor_SMD:CP_Elec_6.3x7.7" (id 2) (at 101.6 74.93 0)
       (effects (font (size 1.27 1.27)) hide)
     )
@@
       (effects (font (size 1.27 1.27)) (justify left))
     )
-    (property "Footprint" "" (id 2) (at 158.75 74.93 0)
+    (property "Footprint" "Capacitor_SMD:CP_Elec_4x5.8" (id 2) (at 158.75 74.93 0)
       (effects (font (size 1.27 1.27)) hide)
     )

Commit message: Fix missing part info
Supports #2.
Parts:
- U2: Digi-Key Part Number (none) -> AP2112K-3.3TRG1DICT-ND; Manufacturer (none) -> Diodes Incorporated; Manufacturer Part Number (none) -> AP2112K-3.3TRG1; Mouser Part Number (none) -> 621-AP2112K-3.3TRG1
Changed lines of the file:
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@@
+      (effects (font (size 1.27 1.27)) hide)
+    )
+    (property "Manufacturer" "Diodes Incorporated" (id 4) (at 139.7 133.35 0)
+      (effects (font (size 1.27 1.27)) hide)
+    )
+    (property "Manufacturer Part Number" "AP2112K-3.3TRG1" (id 5) (at 139.7 133.35 0)
+      (effects (font (size 1.27 1.27)) hide)
+    )
+    (property "Digi-Key Part Number" "AP2112K-3.3TRG1DICT-ND" (id 6) (at 139.7 133.35 0)
+      (effects (font (size 1.27 1.27)) hide)
+    )
+    (property "Mouser Part Number" "621-AP2112K-3.3TRG1" (id 7) (at 139.7 133.35 0)
       (effects (font (size 1.27 1.27)) hide)
     )

Commit message: Replace Digi-Key part numbers with links
Supports #2.
Parts:
- C1: Digi-Key (none) -> https://www.digikey.com/en/products/detail/panasonic-electr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; Digi-Key Part Number PCE3753CT-ND -> (none)
- C2: Digi-Key (none) -> https://www.digikey.com/en/products/detail/kemet/C0603C104M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; Digi-Key Part Number 399-C0603C104M3RAC7867CT-ND -> (none)
- C3: Digi-Key (none) -> https://www.digikey.com/en/products/detail/panasonic-electr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; Digi-Key Part Number 10-EEE-FN1A470URCT-ND -> (none)
- C4, C6: Digi-Key (none) -> https://www.digikey.com/en/products/detail/kemet/C0603C104M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; Digi-Key Part Number 399-C0603C104M8RAC7867CT-ND -> (none)
- C5: Digi-Key (none) -> https://www.digikey.com/en/products/detail/kemet/C0603C106M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; Digi-Key Part Number 399-C0603C106M9PAC7867CT-ND -> (none)
- D1, D2: Digi-Key (none) -> https://www.digikey.com/en/products/detail/onsemi/MBR120LSF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; Digi-Key Part Number MBR120LSFT3GOSCT-ND -> (none)
- D3, D4: Digi-Key (none) -> https://www.digikey.com/en/products/detail/liteon/LTST-C190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; Digi-Key Part Number 160-1435-1-ND -> (none)
- R1, R2: Digi-Key (none) -> https://www.digikey.com/en/products/detail/panasonic-electr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; Digi-Key Part Number P330HCT-ND -> (none)
- U1: Digi-Key (none) -> https://www.digikey.com/en/products/detail/onsemi/NCP1117DT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; Digi-Key Part Number NCP1117DT50RKGOSCT-ND -> (none)
- U2: Digi-Key (none) -> https://www.digikey.com/en/products/detail/diodes-incorpora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; Digi-Key Part Number AP2112K-3.3TRG1DICT-ND -> (none)
Changed lines of the file:
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@@
       (effects (font (size 1.27 1.27)) hide)
     )
-    (property "Digi-Key Part Number" "160-1435-1-ND" (id 6) (at 196.85 74.93 90)
+    (property "Digi-Key" "https://www.digikey.com/en/products/detail/liteon/LTST-C190KGKT/386815" (id 6) (at 196.85 74.93 90)
       (effects (font (size 1.27 1.27)) hide)
     )
@@
       (effects (font (size 1.27 1.27)) hide)
     )
-    (property "Digi-Key Part Number" "P330HCT-ND" (id 6) (at 196.85 85.09 0)
+    (property "Digi-Key" "https://www.digikey.com/en/products/detail/panasonic-electronic-components/ERJ-3EKF3300V/1746374" (id 6) (at 196.85 85.09 0)
       (effects (font (size 1.27 1.27)) hide)
     )
@@
       (effects (font (size 1.27 1.27)) hide)
     )
-    (property "Digi-Key Part Number" "399-C0603C104M8RAC7867CT-ND" (id 6) (at 177.8 135.89 0)
+    (property "Digi-Key" "https://www.digikey.com/en/products/detail/kemet/C0603C104M8RAC7867/2199783" (id 6) (at 177.8 135.89 0)
       (effects (font (size 1.27 1.27)) hide)
     )
@@
       (effects (font (size 1.27 1.27)) hide)
     )
-    (property "Digi-Key Part Number" "NCP1117DT50RKGOSCT-ND" (id 6) (at 139.7 69.85 0)
+    (property "Digi-Key" "https://www.digikey.com/en/products/detail/onsemi/NCP1117DT50RKG/661206" (id 6) (at 139.7 69.85 0)
       (effects (font (size 1.27 1.27)) hide)
     )
@@
       (effects (font (size 1.27 1.27)) hide)
     )
-    (property "Digi-Key Part Number" "PCE3753CT-ND" (id 6) (at 101.6 74.93 0)
+    (property "Digi-Key" "https://www.digikey.com/en/products/detail/panasonic-electronic-components/EEE-HC1E470XP/672769" (id 6) (at 101.6 74.93 0)
       (effects (font (size 1.27 1.27)) hide)
     )
@@
       (effects (font (size 1.27 1.27)) hide)
     )
-    (property "Digi-Key Part Number" "MBR120LSFT3GOSCT-ND" (id 6) (at 82.55 64.77 0)
+    (property "Digi-Key" "https://www.digikey.com/en/products/detail/onsemi/MBR120LSFT3G/1477155" (id 6) (at 82.55 64.77 0)
       (effects (font (size 1.27 1.27)) hide)
     )
@@
       (effects (font (size 1.27 1.27)) hide)
     )
-    (property "Digi-Key Part Number" "10-EEE-FN1A470URCT-ND" (id 6) (at 158.75 74.93 0)
+    (property "Digi-Key" "https://www.digikey.com/en/products/detail/panasonic-electronic-components/EEE-FN1A470UR/11656979" (id 6) (at 158.75 74.93 0)
       (effects (font (size 1.27 1.27)) hide)
     )
@@
       (effects (font (size 1.27 1.27)) hide)
     )
-    (property "Digi-Key Part Number" "399-C0603C104M8RAC7867CT-ND" (id 6) (at 177.8 74.93 0)
+    (property "Digi-Key" "https://www.digikey.com/en/products/detail/kemet/C0603C104M8RAC7867/2199783" (id 6) (at 177.8 74.93 0)
       (effects (font (size 1.27 1.27)) hide)
     )
@@
       (effects (font (size 1.27 1.27)) hide)
     )
-    (property "Digi-Key Part Number" "160-1435-1-ND" (id 6) (at 196.85 135.89 90)
+    (property "Digi-Key" "https://www.digikey.com/en/products/detail/liteon/LTST-C190KGKT/386815" (id 6) (at 196.85 135.89 90)
       (effects (font (size 1.27 1.27)) hide)
     )
@@
       (effects (font (size 1.27 1.27)) hide)
     )
-    (property "Digi-Key Part Number" "399-C0603C104M3RAC7867CT-ND" (id 6) (at 120.65 74.93 0)
+    (property "Digi-Key" "https://www.digikey.com/en/products/detail/kemet/C0603C104M3RAC7867/416046" (id 6) (at 120.65 74.93 0)
       (effects (font (size 1.27 1.27)) hide)
     )
@@
       (effects (font (size 1.27 1.27)) hide)
     )
-    (property "Digi-Key Part Number" "MBR120LSFT3GOSCT-ND" (id 6) (at 153.67 64.77 0)
+    (property "Digi-Key" "https://www.digikey.com/en/products/detail/onsemi/MBR120LSFT3G/1477155" (id 6) (at 153.67 64.77 0)
       (effects (font (size 1.27 1.27)) hide)
     )
@@
       (effects (font (size 1.27 1.27)) hide)
     )
-    (property "Digi-Key Part Number" "P330HCT-ND" (id 6) (at 196.85 146.05 0)
+    (property "Digi-Key" "https://www.digikey.com/en/products/detail/panasonic-electronic-components/ERJ-3EKF3300V/1746374" (id 6) (at 196.85 146.05 0)
       (effects (font (size 1.27 1.27)) hide)
     )
@@
       (effects (font (size 1.27 1.27)) hide)
     )
-    (property "Digi-Key Part Number" "399-C0603C106M9PAC7867CT-ND" (id 6) (at 158.75 135.89 0)
+    (property "Digi-Key" "https://www.digikey.com/en/products/detail/kemet/C0603C106M9PAC7867/1950664" (id 6) (at 158.75 135.89 0)
       (effects (font (size 1.27 1.27)) hide)
     )
@@
       (effects (font (size 1.27 1.27)) hide)
     )
-    (property "Digi-Key Part Number" "AP2112K-3.3TRG1DICT-ND" (id 6) (at 139.7 133.35 0)
-      (effects (font (size 1.27 1.27)) hide)
-    )
+    (property "Digi-Key" "https://www.digikey.com/en/products/detail/diodes-incorporated/AP2112K-3-3TRG1/4470746" (id 6) (at 139.7 133.35 0)
+      (effects (font (size 1.27 1.27)) hide)
+    )

Commit message: Replace Mouser part numbers with links
Supports #2.
Parts:
- C1: Mouser (none) -> https://www.mouser.com/ProductDetail/Panasonic/EEE-HC1E470X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; Mouser Part Number 667-EEE-HC1E470XP -> (none)
- C2: Mouser (none) -> https://www.mouser.com/ProductDetail/KEMET/C0603C104M3RAC?q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; Mouser Part Number 80-C0603C104M3RAC -> (none)
- C3: Mouser (none) -> https://www.mouser.com/ProductDetail/Panasonic/EEE-FN1A470U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; Mouser Part Number 667-EEE-FN1A470UR -> (none)
- C4, C6: Mouser (none) -> https://www.mouser.com/ProductDetail/KEMET/C0603C104M8RACTU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; Mouser Part Number 80-C0603C104M8R -> (none)
- C5: Mouser (none) -> https://www.mouser.com/ProductDetail/KEMET/C0603C106M9PAC?q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; Mouser Part Number 80-C0603C106M9PAC -> (none)
- D1, D2: Mouser (none) -> https://www.mouser.com/ProductDetail/onsemi/MBR120LSFT3G?qs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; Mouser Part Number 863-MBR120LSFT3G -> (none)
- D3, D4: Mouser (none) -> https://www.mouser.com/ProductDetail/Lite-On/LTST-C190KGKT?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; Mouser Part Number 859-LTST-C190KGKT -> (none)
- R1, R2: Mouser (none) -> https://www.mouser.com/ProductDetail/Panasonic/ERJ-3EKF3300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; Mouser Part Number 667-ERJ-3EKF3300V -> (none)
- U1: Mouser (none) -> https://www.mouser.com/ProductDetail/onsemi/NCP1117DT50RKG?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; Mouser Part Number 863-NCP1117DT50RKG -> (none)
- U2: Mouser (none) -> https://www.mouser.com/ProductDetail/Diodes-Incorporated/AP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; Mouser Part Number 621-AP2112K-3.3TRG1 -> (none)
Changed lines of the file:
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@@
       (effects (font (size 1.27 1.27)) hide)
     )
-    (property "Mouser Part Number" "859-LTST-C190KGKT" (id 7) (at 196.85 74.93 90)
+    (property "Mouser" "https://www.mouser.com/ProductDetail/Lite-On/LTST-C190KGKT?qs=205qCy6M2Q%252BAdcgwUZktqw%3D%3D" (id 7) (at 196.85 74.93 90)
       (effects (font (size 1.27 1.27)) hide)
     )
@@
       (effects (font (size 1.27 1.27)) hide)
     )
-    (property "Mouser Part Number" "667-ERJ-3EKF3300V" (id 7) (at 196.85 85.09 0)
+    (property "Mouser" "https://www.mouser.com/ProductDetail/Panasonic/ERJ-3EKF3300V?qs=MVjVSMjNRMqskx0rzM4%2FYg%3D%3D" (id 7) (at 196.85 85.09 0)
       (effects (font (size 1.27 1.27)) hide)
     )
@@
       (effects (font (size 1.27 1.27)) hide)
     )
-    (property "Mouser Part Number" "80-C0603C104M8R" (id 7) (at 177.8 135.89 0)
+    (property "Mouser" "https://www.mouser.com/ProductDetail/KEMET/C0603C104M8RACTU?qs=t9q%2F2xDdjt%252BO6KYorkYlEw%3D%3D" (id 7) (at 177.8 135.89 0)
       (effects (font (size 1.27 1.27)) hide)
     )
@@
       (effects (font (size 1.27 1.27)) hide)
     )
-    (property "Mouser Part Number" "863-NCP1117DT50RKG" (id 7) (at 139.7 69.85 0)
+    (property "Mouser" "https://www.mouser.com/ProductDetail/onsemi/NCP1117DT50RKG?qs=Gev%252BmEvV0iaGLyZQ1w6kFw%3D%3D" (id 7) (at 139.7 69.85 0)
       (effects (font (size 1.27 1.27)) hide)
     )
@@
       (effects (font (size 1.27 1.27)) hide)
     )
-    (property "Mouser Part Number" "667-EEE-HC1E470XP" (id 7) (at 101.6 74.93 0)
+    (property "Mouser" "https://www.mouser.com/ProductDetail/Panasonic/EEE-HC1E470XP?qs=Ywefl8B65e6qyZdKUyDlkQ%3D%3D" (id 7) (at 101.6 74.93 0)
       (effects (font (size 1.27 1.27)) hide)
     )
@@
       (effects (font (size 1.27 1.27)) hide)
     )
-    (property "Mouser Part Number" "863-MBR120LSFT3G" (id 7) (at 82.55 64.77 0)
+    (property "Mouser" "https://www.mouser.com/ProductDetail/onsemi/MBR120LSFT3G?qs=3JMERSakebrl0QzFyBgvHg%3D%3D" (id 7) (at 82.55 64.77 0)
       (effects (font (size 1.27 1.27)) hide)
     )
@@
       (effects (font (size 1.27 1.27)) hide)
     )
-    (property "Mouser Part Number" "667-EEE-FN1A470UR" (id 7) (at 158.75 74.93 0)
+    (property "Mouser" "https://www.mouser.com/ProductDetail/Panasonic/EEE-FN1A470UR?qs=OlC7AqGiEDlZjloUmme03Q%3D%3D" (id 7) (at 158.75 74.93 0)
       (effects (font (size 1.27 1.27)) hide)
     )
@@
       (effects (font (size 1.27 1.27)) hide)
     )
-    (property "Mouser Part Number" "80-C0603C104M8R" (id 7) (at 177.8 74.93 0)
+    (property "Mouser" "https://www.mouser.com/ProductDetail/KEMET/C0603C104M8RACTU?qs=t9q%2F2xDdjt%252BO6KYorkYlEw%3D%3D" (id 7) (at 177.8 74.93 0)
       (effects (font (size 1.27 1.27)) hide)
     )
@@
       (effects (font (size 1.27 1.27)) hide)
     )
-    (property "Mouser Part Number" "859-LTST-C190KGKT" (id 7) (at 196.85 135.89 90)
+    (property "Mouser" "https://www.mouser.com/ProductDetail/Lite-On/LTST-C190KGKT?qs=205qCy6M2Q%252BAdcgwUZktqw%3D%3D" (id 7) (at 196.85 135.89 90)
       (effects (font (size 1.27 1.27)) hide)
     )
@@
       (effects (font (size 1.27 1.27)) hide)
     )
-    (property "Mouser Part Number" "80-C0603C104M3RAC" (id 7) (at 120.65 74.93 0)
+    (property "Mouser" "https://www.mouser.com/ProductDetail/KEMET/C0603C104M3RAC?qs=zlI8QACJnq99iivvUDrLjA%3D%3D" (id 7) (at 120.65 74.93 0)
       (effects (font (size 1.27 1.27)) hide)
     )
@@
       (effects (font (size 1.27 1.27)) hide)
     )
-    (property "Mouser Part Number" "863-MBR120LSFT3G" (id 7) (at 153.67 64.77 0)
+    (property "Mouser" "https://www.mouser.com/ProductDetail/onsemi/MBR120LSFT3G?qs=3JMERSakebrl0QzFyBgvHg%3D%3D" (id 7) (at 153.67 64.77 0)
       (effects (font (size 1.27 1.27)) hide)
     )
@@
       (effects (font (size 1.27 1.27)) hide)
     )
-    (property "Mouser Part Number" "667-ERJ-3EKF3300V" (id 7) (at 196.85 146.05 0)
+    (property "Mouser" "https://www.mouser.com/ProductDetail/Panasonic/ERJ-3EKF3300V?qs=MVjVSMjNRMqskx0rzM4%2FYg%3D%3D" (id 7) (at 196.85 146.05 0)
       (effects (font (size 1.27 1.27)) hide)
     )
@@
       (effects (font (size 1.27 1.27)) hide)
     )
-    (property "Mouser Part Number" "80-C0603C106M9PAC" (id 7) (at 158.75 135.89 0)
+    (property "Mouser" "https://www.mouser.com/ProductDetail/KEMET/C0603C106M9PAC?qs=vnwGVgFuQibgQzzOtLArWQ%3D%3D" (id 7) (at 158.75 135.89 0)
       (effects (font (size 1.27 1.27)) hide)
     )
@@
       (effects (font (size 1.27 1.27)) hide)
     )
-    (property "Mouser Part Number" "621-AP2112K-3.3TRG1" (id 7) (at 139.7 133.35 0)
-      (effects (font (size 1.27 1.27)) hide)
-    )
+    (property "Mouser" "https://www.mouser.com/ProductDetail/Diodes-Incorporated/AP2112K-3.3TRG1?qs=x6A8l6qLYDDPYHosCdzh%2FA%3D%3D" (id 7) (at 139.7 133.35 0)
+      (effects (font (size 1.27 1.27)) hide)
+    )
