File: pcb-main-nautilus-atmega4809.kicad_pcb (KiCad board)
At the start: 2 copper layers, 110 parts, among them J1 694106301002, J2 105017-0001, J3 FTSH-105-01-L-DV-007-K, J4 75844-101-06LF, J5 66951-006LF, J6 66951-010LF, J7 66951-008LF, J8 66951-008LF, Q1 BSS138PW, Q2 BSS138PW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

Commit message: Configure board stackup
Supports #4.
Other:
- copper layers 2 -> 4
Changed lines of the file:
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@@
 (kicad_pcb (version 20211014) (generator pcbnew)
   (general
-    (thickness 1.6)
+    (thickness 1.567)
   )
   (paper "A")
@@
   (layers
     (0 "F.Cu" signal)
+    (1 "In1.Cu" power)
+    (2 "In2.Cu" power)
     (31 "B.Cu" signal)
     (32 "B.Adhes" user "B.Adhesive")
@@
   (setup
     (stackup
-      (layer "F.SilkS" (type "Top Silk Screen"))
+      (layer "F.SilkS" (type "Top Silk Screen") (color "White"))
       (layer "F.Paste" (type "Top Solder Paste"))
-      (layer "F.Mask" (type "Top Solder Mask") (thickness 0.01))
-      (layer "F.Cu" (type "copper") (thickness 0.035))
-      (layer "dielectric 1" (type "core") (thickness 1.51) (material "FR4") (epsilon_r 4.5) (loss_tangent 0.02))
-      (layer "B.Cu" (type "copper") (thickness 0.035))
-      (layer "B.Mask" (type "Bottom Solder Mask") (thickness 0.01))
+      (layer "F.Mask" (type "Top Solder Mask") (color "Purple") (thickness 0.0254))
+      (layer "F.Cu" (type "copper") (thickness 0.0432))
+      (layer "dielectric 1" (type "core") (thickness 0.2021) (material "FR4") (epsilon_r 4.5) (loss_tangent 0.02))
+      (layer "In1.Cu" (type "copper") (thickness 0.0175))
+      (layer "dielectric 2" (type "prepreg") (thickness 0.9906) (material "FR4") (epsilon_r 4.5) (loss_tangent 0.02))
+      (layer "In2.Cu" (type "copper") (thickness 0.0175))
+      (layer "dielectric 3" (type "core") (thickness 0.2021) (material "FR4") (epsilon_r 4.5) (loss_tangent 0.02))
+      (layer "B.Cu" (type "copper") (thickness 0.0432))
+      (layer "B.Mask" (type "Bottom Solder Mask") (color "Purple") (thickness 0.0254))
       (layer "B.Paste" (type "Bottom Solder Paste"))
-      (layer "B.SilkS" (type "Bottom Silk Screen"))
+      (layer "B.SilkS" (type "Bottom Silk Screen") (color "White"))
       (copper_finish "None")
       (dielectric_constraints no)

Commit message: Configure constraints
Supports #4.
Other:
- rule pad_to_mask_clearance: 0 -> 0.0508
Changed lines of the file:
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@@
       (layer "B.Paste" (type "Bottom Solder Paste"))
       (layer "B.SilkS" (type "Bottom Silk Screen") (color "White"))
-      (copper_finish "None")
       (dielectric_constraints no)
     )
-    (pad_to_mask_clearance 0)
+    (pad_to_mask_clearance 0.0508)
+    (solder_mask_min_width 0.1016)
     (pcbplotparams
       (layerselection 0x00010fc_ffffffff)

Commit message: Fix use of wrong symbol
Supports #4.
Parts:
- moved J1 1.95 mm to (88.9, 91.4)
Connections:
- J1 pad 3: (no net) -> /GND
Changed lines of the file:
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@@
       (layer "B.Paste" (type "Bottom Solder Paste"))
       (layer "B.SilkS" (type "Bottom Silk Screen") (color "White"))
+      (copper_finish "None")
       (dielectric_constraints no)
     )
@@
     )
   )
+  (footprint "Connector_BarrelJack:BarrelJack_Wuerth_6941xx301002" (layer "F.Cu")
+    (at 88.9 91.44)
+    (descr "Wuerth electronics barrel jack connector (5.5mm outher diameter, inner diameter 2.05mm or 2.55mm depending on exact order number), See: http://katalog.we-online.de/em/datasheet/6941xx301002.pdf")
+    (tags "connector barrel jack")
+    (property "Digi-Key Part Number" "732-5930-ND")
+    (property "Manufacturer" "Würth Elektronik")
+    (property "Manufacturer Part Number" "694106301002")
+    (property "Mouser Part Number" "710-694106301002")
+    (property "Sheetfile" "pcb-main-nautilus-atmega4809.kicad_sch")
+    (property "Sheetname" "")
+    (attr through_hole)
+    (fp_text reference "J1" (at 0 -2.5) (layer "F.SilkS")
+      (effects (font (size 1 1) (thickness 0.15)))
+    )
+    (fp_text value "694106301002" (at 0 15.5) (layer "F.Fab")
+      (effects (font (size 1 1) (thickness 0.15)))
+    )
+    (fp_text user "${REFERENCE}" (at 0 7.5) (layer "F.Fab")
+      (effects (font (size 1 1) (thickness 0.15)))
+    )
+    (fp_line (start -4.6 13.7) (end -4.6 -1) (layer "F.SilkS") (width 0.12))
+    (fp_line (start 4.6 13.7) (end -4.6 13.7) (layer "F.SilkS") (width 0.12))
+    (fp_line (start -4.6 -1) (end -2.5 -1) (layer "F.SilkS") (width 0.12))
+    (fp_line (start 4.6 -1) (end 4.6 0.8) (layer "F.SilkS") (width 0.12))
+    (fp_line (start -3.2 -1.3) (end -4.9 -1.3) (layer "F.SilkS") (width 0.12))
+    (fp_line (start 2.5 -1) (end 4.6 -1) (layer "F.SilkS") (width 0.12))
+    (fp_line (start -4.9 -1.3) (end -4.9 0.3) (layer "F.SilkS") (width 0.12))
+    (fp_line (start 4.6 5.2) (end 4.6 13.7) (layer "F.SilkS") (width 0.12))
+    (fp_line (start 5 -1.4) (end -5 -1.4) (layer "F.CrtYd") (width 0.05))
+    (fp_line (start -5 -1.4) (end -5 14.1) (layer "F.CrtYd") (width 0.05))
+    (fp_line (start 6.2 0.5) (end 5 0.5) (layer "F.CrtYd") (width 0.05))
+    (fp_line (start 6.2 5.5) (end 5 5.5) (layer "F.CrtYd") (width 0.05))
+    (fp_line (start 6.2 0.5) (end 6.2 5.5) (layer "F.CrtYd") (width 0.05))
+    (fp_line (start 5 0.5) (end 5 -1.4) (layer "F.CrtYd") (width 0.05))
+    (fp_line (start 5 14.1) (end 5 5.5) (layer "F.CrtYd") (width 0.05))
+    (fp_line (start -5 14.1) (end 5 14.1) (layer "F.CrtYd") (width 0.05))
+    (fp_line (start -4.5 0.1) (end -3.5 -0.9) (layer "F.Fab") (width 0.1))
+    (fp_line (start 4.5 -0.9) (end 4.5 13.6) (layer "F.Fab") (width 0.1))
+    (fp_line (start -4.5 13.6) (end -4.5 0.1) (layer "F.Fab") (width 0.1))
+    (fp_line (start 4.5 -0.9) (end -3.5 -0.9) (layer "F.Fab") (width 0.1))
+    (fp_line (start 4.5 13.6) (end -4.5 13.6) (layer "F.Fab") (width 0.1))
+    (pad "1" thru_hole rect (at 0 0) (size 4.4 1.8) (drill oval 3.4 0.8) (layers *.Cu *.Mask)
+      (net 12 "/POWER/PWRIN") (pintype "passive"))
+    (pad "2" thru_hole oval (at 0 5.8) (size 4 1.8) (drill oval 3 0.8) (layers *.Cu *.Mask)
+      (net 2 "/GND") (pintype "passive"))
+    (pad "3" thru_hole oval (at 4.8 3 90) (size 4 1.8) (drill oval 3 0.8) (layers *.Cu *.Mask)
+      (net 2 "/GND") (pintype "passive"))
+    (model "${KICAD6_3DMODEL_DIR}/Connector_BarrelJack.3dshapes/BarrelJack_Wuerth_6941xx301002.wrl"
+      (offset (xyz 0 0 0))
+      (scale (xyz 1 1 1))
+      (rotate (xyz 0 0 0))
+    )
+  )
   (footprint "Connector_PinHeader_2.54mm:PinHeader_2x03_P2.54mm_Vertical" (layer "F.Cu")
     (at 98.98 90.18)
@@
       (offset (xyz 0 0 0))
       (scale (xyz 1 1 1))
-      (rotate (xyz 0 0 0))
-    )
-  )
-  (footprint "Connector_BarrelJack:BarrelJack_Wuerth_6941xx301002" (layer "F.Cu")
-    (at 89.93 89.78)
-    (descr "Wuerth electronics barrel jack connector (5.5mm outher diameter, inner diameter 2.05mm or 2.55mm depending on exact order number), See: http://katalog.we-online.de/em/datasheet/6941xx301002.pdf")
-    (tags "connector barrel jack")
-    (property "Digi-Key Part Number" "732-5930-ND")
-    (property "Manufacturer" "Würth Elektronik")
-    (property "Manufacturer Part Number" "694106301002")
-    (property "Mouser Part Number" "710-694106301002")
-    (property "Sheetfile" "pcb-main-nautilus-atmega4809.kicad_sch")
-    (property "Sheetname" "")
-    (attr through_hole)
-    (fp_text reference "J1" (at 0 -2.5) (layer "F.SilkS")
-      (effects (font (size 1 1) (thickness 0.15)))
-    )
-    (fp_text value "694106301002" (at 0 15.5) (layer "F.Fab")
-      (effects (font (size 1 1) (thickness 0.15)))
-    )
-    (fp_text user "${REFERENCE}" (at 0 7.5) (layer "F.Fab")
-      (effects (font (size 1 1) (thickness 0.15)))
-    )
-    (fp_line (start -4.6 -1) (end -2.5 -1) (layer "F.SilkS") (width 0.12))
-    (fp_line (start 4.6 -1) (end 4.6 0.8) (layer "F.SilkS") (width 0.12))
-    (fp_line (start 4.6 13.7) (end -4.6 13.7) (layer "F.SilkS") (width 0.12))
-    (fp_line (start 4.6 5.2) (end 4.6 13.7) (layer "F.SilkS") (width 0.12))
-    (fp_line (start -4.6 13.7) (end -4.6 -1) (layer "F.SilkS") (width 0.12))
-    (fp_line (start -4.9 -1.3) (end -4.9 0.3) (layer "F.SilkS") (width 0.12))
-    (fp_line (start -3.2 -1.3) (end -4.9 -1.3) (layer "F.SilkS") (width 0.12))
-    (fp_line (start 2.5 -1) (end 4.6 -1) (layer "F.SilkS") (width 0.12))
-    (fp_line (start 5 14.1) (end 5 5.5) (layer "F.CrtYd") (width 0.05))
-    (fp_line (start 5 -1.4) (end -5 -1.4) (layer "F.CrtYd") (width 0.05))
-    (fp_line (start 6.2 0.5) (end 5 0.5) (layer "F.CrtYd") (width 0.05))
-    (fp_line (start 6.2 0.5) (end 6.2 5.5) (layer "F.CrtYd") (width 0.05))
-    (fp_line (start -5 14.1) (end 5 14.1) (layer "F.CrtYd") (width 0.05))
-    (fp_line (start -5 -1.4) (end -5 14.1) (layer "F.CrtYd") (width 0.05))
-    (fp_line (start 5 0.5) (end 5 -1.4) (layer "F.CrtYd") (width 0.05))
-    (fp_line (start 6.2 5.5) (end 5 5.5) (layer "F.CrtYd") (width 0.05))
-    (fp_line (start -4.5 13.6) (end -4.5 0.1) (layer "F.Fab") (width 0.1))
-    (fp_line (start 4.5 -0.9) (end 4.5 13.6) (layer "F.Fab") (width 0.1))
-    (fp_line (start 4.5 -0.9) (end -3.5 -0.9) (layer "F.Fab") (width 0.1))
-    (fp_line (start -4.5 0.1) (end -3.5 -0.9) (layer "F.Fab") (width 0.1))
-    (fp_line (start 4.5 13.6) (end -4.5 13.6) (layer "F.Fab") (width 0.1))
-    (pad "1" thru_hole rect (at 0 0) (size 4.4 1.8) (drill oval 3.4 0.8) (layers *.Cu *.Mask)
-      (net 12 "/POWER/PWRIN") (pintype "passive"))
-    (pad "2" thru_hole oval (at 0 5.8) (size 4 1.8) (drill oval 3 0.8) (layers *.Cu *.Mask)
-      (net 2 "/GND") (pintype "passive"))
-    (pad "3" thru_hole oval (at 4.8 3 90) (size 4 1.8) (drill oval 3 0.8) (layers *.Cu *.Mask))
-    (model "${KICAD6_3DMODEL_DIR}/Connector_BarrelJack.3dshapes/BarrelJack_Wuerth_6941xx301002.wrl"
-      (offset (xyz 0 0 0))
-      (scale (xyz 1 1 1))

Commit message: Move components to edge of work area
Supports #4.
Parts:
- moved C1 81.7 mm to (52.7, 31.8)
- moved C10 81.7 mm to (65.1, 57.2)
- moved C11 81.7 mm to (37.4, 64.8)
- moved C12 81.7 mm to (41.8, 59.7)
- moved C13 81.7 mm to (37.4, 59.8)
- moved C14 81.7 mm to (33.0, 64.8)
- moved C16 81.7 mm to (33.0, 59.8)
- moved C17 81.7 mm to (33.0, 62.3)
- moved C2 81.7 mm to (85.3, 32.7)
- moved C5 81.7 mm to (86.7, 41.4)
- moved C6 81.7 mm to (92.7, 35.7)
- moved C7 81.7 mm to (98.2, 27.6)
- moved C9 81.7 mm to (65.1, 59.7)
- moved D1 81.7 mm to (21.6, 50.3)
- moved D2 81.7 mm to (82.9, 38.4)
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
Commit message: Add board outline
Supports #4.
Other:
- board outline added: 68.6 x 53.3 mm
Changed lines of the file:
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@@
       (net 4 "/5V") (pinfunction "1") (pintype "passive"))
   )
+  (gr_line (start 164.516 96.66) (end 166.04 98.184) (layer "Edge.Cuts") (width 0.254))
+  (gr_line (start 166.04 109.614) (end 168.58 112.154) (layer "Edge.Cuts") (width 0.254))
+  (gr_line (start 166.04 147.46) (end 168.58 144.92) (layer "Edge.Cuts") (width 0.254))
+  (gr_arc (start 166.04 149) (mid 165.747107 149.707107) (end 165.04 150) (layer "Edge.Cuts") (width 0.254))
+  (gr_line (start 165.04 150) (end 101 150) (layer "Edge.Cuts") (width 0.254))
+  (gr_line (start 101 96.66) (end 164.516 96.66) (layer "Edge.Cuts") (width 0.254))
+  (gr_arc (start 101 150) (mid 100.292893 149.707107) (end 100 149) (layer "Edge.Cuts") (width 0.254))
+  (gr_line (start 166.04 98.184) (end 166.04 109.614) (layer "Edge.Cuts") (width 0.254))
+  (gr_line (start 166.04 147.46) (end 166.04 149) (layer "Edge.Cuts") (width 0.254))
+  (gr_line (start 100 149) (end 100 97.66) (layer "Edge.Cuts") (width 0.254))
+  (gr_line (start 168.58 144.92) (end 168.58 112.154) (layer "Edge.Cuts") (width 0.254))
+  (gr_arc (start 100 97.66) (mid 100.292893 96.952893) (end 101 96.66) (layer "Edge.Cuts") (width 0.254))
 )

Commit message: Place headers and power connector
Supports #4.
Parts:
- moved J5 178.4 mm to (163.5, 147.5), turned to -90 degrees
- moved J8 172.5 mm to (145.7, 147.5), turned to -90 degrees
- moved J4 147.2 mm to (163.6, 119.5)
- moved J7 137.7 mm to (145.7, 99.2), turned to 90 degrees
- moved J1 136.0 mm to (111.1, 141.6), turned to -90 degrees
- moved J6 123.4 mm to (118.8, 99.2), turned to 90 degrees
