File: pcb-main-nautilus-atmega4809.kicad_pcb (KiCad board)
At the start: 4 copper layers, 68.6 x 53.3 mm, 91 parts, among them J1 694106301002, J2 105017-0001, J3 FTSH-105-01-L-DV-007-K, J4 75844-101-06LF, J5 66951-006LF, J6 66951-010LF, J7 66951-008LF, J8 66951-008LF, Q1 BSS138PW, Q2 BSS138PW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

Commit message: Add board info silk
Supports #4.
Other:
- board text added: "VERSION: ${REVISION}"
- board text added: "https://github.com/apcountryman/pcb-main-nautilus-atmega4809"
Changed lines of the file:
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@@
   (gr_line locked (start 168.58 144.92) (end 168.58 112.154) (layer "Edge.Cuts") (width 0.1))
   (gr_arc locked (start 100 97.66) (mid 100.292893 96.952893) (end 101 96.66) (layer "Edge.Cuts") (width 0.1))
+  (gr_text "VERSION: ${REVISION}" (at 164.5 103.5) (layer "B.SilkS")
+    (effects (font (size 1 1) (thickness 0.15)) (justify left mirror))
+  )
+  (gr_text "https://github.com/apcountryman/pcb-main-nautilus-atmega4809" (at 164.5 101.5) (layer "B.SilkS")
+    (effects (font (size 1 1) (thickness 0.15)) (justify left mirror))
+  )
   (gr_text "D2" (at 158.42 100.5 270) (layer "F.SilkS")
     (effects (font (size 1 1) (thickness 0.15)) (justify left))
