File: pcb-main-nautilus-atmega4809-sheet-updi_programmer_and_usb_serial_bridge.kicad_sch (KiCad schematic)
At the start: 6 parts, among them U3 ATSAMD11D14A-SS

Commit message: Address review findings
Supports #2.
Parts:
- U3: Manufacturer Part Number ATSAMD11D14A-SS -> ATSAMD11D14A-SSU
Changed lines of the file:
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@@
     (title "https://github.com/apcountryman/pcb-main-nautilus-atmega4809")
     (rev "GIT_VERSION")
-    (comment 1 "Derivative of the \"Arduino UNO Rev3\" (https://docs.arduino.cc/hardware/uno-rev3) and\\n\"Arduino Nano Every\" (https://docs.arduino.cc/hardware/nano-every) reference designs")
+    (comment 1 "Derivative of the \"Arduino UNO Rev3\" (https://docs.arduino.cc/hardware/uno-rev3) and\\n\"Arduino Nano Every\" (https://docs.arduino.cc/hardware/nano-every) reference designs.")
   )
   (junction (at 96.52 91.44) (diameter 0) (color 0 0 0 0)
@@
       (effects (font (size 1.27 1.27)) hide)
     )
-    (property "Manufacturer Part Number" "ATSAMD11D14A-SS" (id 5) (at 139.7 101.6 0)
-      (effects (font (size 1.27 1.27)) hide)
-    )
+    (property "Manufacturer Part Number" "ATSAMD11D14A-SSU" (id 5) (at 139.7 101.6 0)
+      (effects (font (size 1.27 1.27)) hide)
+    )

Commit message: Add missing test points
Supports #4.
Parts:
- added TP49, TP50, TP51: TestPoint, TestPoint:TestPoint_Pad_D1.0mm, symbol Connector:TestPoint
Connections:
- net BI-DIRECTIONAL LEVEL SHIFTER: RX/SIGNAL_3.3V: now also TP49.1
- net BI-DIRECTIONAL LEVEL SHIFTER: TX/SIGNAL_3.3V: now also TP50.1
- net BI-DIRECTIONAL LEVEL SHIFTER: UPDI/SIGNAL_3.3V: now also TP51.1
Changed lines of the file:
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@@
   (junction (at 139.7 73.66) (diameter 0) (color 0 0 0 0)
   )
+  (junction (at 162.56 101.6) (diameter 0) (color 0 0 0 0)
+  )
+  (junction (at 162.56 121.92) (diameter 0) (color 0 0 0 0)
+  )
   (junction (at 139.7 63.5) (diameter 0) (color 0 0 0 0)
+  )
+  (junction (at 160.02 142.24) (diameter 0) (color 0 0 0 0)
   )
   (junction (at 111.76 96.52) (diameter 0) (color 0 0 0 0)
@@
     (stroke (width 0) (type default) (color 0 0 0 0))
   )
+  (wire (pts (xy 157.48 147.32) (xy 162.56 147.32))
+    (stroke (width 0) (type default) (color 0 0 0 0))
+  )
   (wire (pts (xy 93.98 96.52) (xy 111.76 96.52))
     (stroke (width 0) (type default) (color 0 0 0 0))
@@
     (stroke (width 0) (type default) (color 0 0 0 0))
   )
+  (wire (pts (xy 160.02 142.24) (xy 172.72 142.24))
+    (stroke (width 0) (type default) (color 0 0 0 0))
+  )
   (wire (pts (xy 200.66 121.92) (xy 203.2 121.92))
     (stroke (width 0) (type default) (color 0 0 0 0))
@@
     (stroke (width 0) (type default) (color 0 0 0 0))
   )
+  (wire (pts (xy 162.56 147.32) (xy 162.56 121.92))
+    (stroke (width 0) (type default) (color 0 0 0 0))
+  )
   (wire (pts (xy 139.7 60.96) (xy 139.7 63.5))
     (stroke (width 0) (type default) (color 0 0 0 0))
@@
     (stroke (width 0) (type default) (color 0 0 0 0))
   )
+  (wire (pts (xy 162.56 101.6) (xy 172.72 101.6))
+    (stroke (width 0) (type default) (color 0 0 0 0))
+  )
+  (wire (pts (xy 157.48 144.78) (xy 160.02 144.78))
+    (stroke (width 0) (type default) (color 0 0 0 0))
+  )
   (wire (pts (xy 152.4 104.14) (xy 154.94 104.14))
     (stroke (width 0) (type default) (color 0 0 0 0))
   )
-  (wire (pts (xy 160.02 142.24) (xy 172.72 142.24))
+  (wire (pts (xy 162.56 99.06) (xy 162.56 101.6))
     (stroke (width 0) (type default) (color 0 0 0 0))
   )
@@
     (stroke (width 0) (type default) (color 0 0 0 0))
   )
-  (wire (pts (xy 154.94 101.6) (xy 172.72 101.6))
+  (wire (pts (xy 154.94 101.6) (xy 162.56 101.6))
     (stroke (width 0) (type default) (color 0 0 0 0))
   )
@@
   )
   (wire (pts (xy 152.4 101.6) (xy 154.94 101.6))
+    (stroke (width 0) (type default) (color 0 0 0 0))
+  )
+  (wire (pts (xy 160.02 144.78) (xy 160.02 142.24))
     (stroke (width 0) (type default) (color 0 0 0 0))
   )
@@
     (pin "2")
   )
+  (symbol (lib_id "Connector:TestPoint") (at 157.48 147.32 90) (unit 1)
+    (in_bom yes) (on_board yes)
+    (property "Reference" "TP50" (id 0) (at 152.4 147.32 90)
+      (effects (font (size 1.27 1.27)) (justify left))
+    )
+    (property "Value" "TestPoint" (id 1) (at 155.4479 144.78 0)
+      (effects (font (size 1.27 1.27)) (justify left) hide)
+    )
+    (property "Footprint" "TestPoint:TestPoint_Pad_D1.0mm" (id 2) (at 157.48 142.24 0)
+      (effects (font (size 1.27 1.27)) hide)
+    )
+    (property "Datasheet" "~" (id 3) (at 157.48 142.24 0)
+      (effects (font (size 1.27 1.27)) hide)
+    )
+    (pin "1")
+  )
+  (symbol (lib_id "Connector:TestPoint") (at 162.56 99.06 0) (unit 1)
+    (in_bom yes) (on_board yes)
+    (property "Reference" "TP51" (id 0) (at 162.56 93.98 90)
+      (effects (font (size 1.27 1.27)) (justify left))
+    )
+    (property "Value" "TestPoint" (id 1) (at 165.1 97.0279 0)
+      (effects (font (size 1.27 1.27)) (justify left) hide)
+    )
+    (property "Footprint" "TestPoint:TestPoint_Pad_D1.0mm" (id 2) (at 167.64 99.06 0)
+      (effects (font (size 1.27 1.27)) hide)
+    )
+    (property "Datasheet" "~" (id 3) (at 167.64 99.06 0)
+      (effects (font (size 1.27 1.27)) hide)
+    )
+    (pin "1")
+  )
+  (symbol (lib_id "Connector:TestPoint") (at 157.48 144.78 90) (unit 1)
+    (in_bom yes) (on_board yes)
+    (property "Reference" "TP49" (id 0) (at 152.4 144.78 90)
+      (effects (font (size 1.27 1.27)) (justify left))
+    )
+    (property "Value" "TestPoint" (id 1) (at 155.4479 142.24 0)
+      (effects (font (size 1.27 1.27)) (justify left) hide)
+    )
+    (property "Footprint" "TestPoint:TestPoint_Pad_D1.0mm" (id 2) (at 157.48 139.7 0)
+      (effects (font (size 1.27 1.27)) hide)
+    )
+    (property "Datasheet" "~" (id 3) (at 157.48 139.7 0)
+      (effects (font (size 1.27 1.27)) hide)
+    )
+    (pin "1")
+  )
   (symbol (lib_id "Device:C_Small") (at 132.08 73.66 270) (unit 1)

Commit message: Remove unnecessary test points
Supports #4.
Parts:
- renumbered TP49 to TP27, TP50 to TP28, TP51 to TP29
Changed lines of the file:
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@@
   (symbol (lib_id "Connector:TestPoint") (at 157.48 147.32 90) (unit 1)
     (in_bom yes) (on_board yes)
-    (property "Reference" "TP50" (id 0) (at 152.4 147.32 90)
+    (property "Reference" "TP28" (id 0) (at 152.4 147.32 90)
       (effects (font (size 1.27 1.27)) (justify left))
     )
@@
   (symbol (lib_id "Connector:TestPoint") (at 162.56 99.06 0) (unit 1)
     (in_bom yes) (on_board yes)
-    (property "Reference" "TP51" (id 0) (at 162.56 93.98 90)
+    (property "Reference" "TP29" (id 0) (at 162.56 93.98 90)
       (effects (font (size 1.27 1.27)) (justify left))
     )
@@
   (symbol (lib_id "Connector:TestPoint") (at 157.48 144.78 90) (unit 1)
     (in_bom yes) (on_board yes)
-    (property "Reference" "TP49" (id 0) (at 152.4 144.78 90)
+    (property "Reference" "TP27" (id 0) (at 152.4 144.78 90)
       (effects (font (size 1.27 1.27)) (justify left))
     )
